Commit message: finished planned urdf (added the lidar and camera with its rotator)

File: install/r2d2_main/share/r2d2_main/urdf/robot.urdf (robot description, URDF)
Before this commit: robot r2d2, 5 links, 4 joints
Links:
- added link camera_link; collision box size=0.04 0.04 0.04; visual box size=0.04 0.04 0.04
- added link camera_rotator_link; collision cylinder length=0.08 radius=0.02; visual cylinder length=0.08 radius=0.02
- added link lidar_link; collision box size=0.08 0.08 0.08; visual box size=0.08 0.08 0.08
Joints:
- added joint camera_joint: type fixed, parent camera_rotator_link, child camera_link, origin xyz=0.05 0 0 rpy=0 0 0
- added joint lidar_joint: type fixed, parent robot_base, child lidar_link, origin xyz=0 0 0.54 rpy=0 0 0
- added joint rotator_joint: type continuous, parent lidar_link, child camera_rotator_link, origin xyz=0 0 0.08 rpy=0 0 0, axis 0 0 1
- joint left_wheel2_joint: axis 0 1 0 -> 0 0 1
- joint right_wheel1_joint: axis 0 1 0 -> 0 0 1
- joint right_wheel2_joint: axis 0 1 0 -> 0 0 1

Commit message: added gazebo plugins and launch files

File: install/r2d2_main/share/r2d2_main/urdf/robot.urdf (robot description, URDF)
Before this commit: robot r2d2, 8 links, 7 joints
Links:
- link camera_link: mass None -> 0.05
- link camera_rotator_link: mass None -> 0.05
- link left_wheel1: mass None -> 0.3; geometry collision cylinder length=0.035 radius=0.049; visual cylinder length=0.035 radius=0.049
- link left_wheel2: mass None -> 0.3; geometry collision cylinder length=0.035 radius=0.049; visual cylinder length=0.035 radius=0.049
- link lidar_link: mass None -> 0.1
- link right_wheel1: mass None -> 0.3; geometry collision cylinder length=0.035 radius=0.049; visual cylinder length=0.035 radius=0.049
- link right_wheel2: mass None -> 0.3; geometry collision cylinder length=0.035 radius=0.049; visual cylinder length=0.035 radius=0.049
- link robot_base: mass None -> 3.0; geometry collision box size=0.28 0.28 0.35; visual box size=0.28 0.28 0.35
Joints:
- joint left_wheel1_joint: origin xyz=-0.1 0.22 0 rpy=-1.5707 0 0 -> xyz=-0.07 0.154 0 rpy=-1.5707 0 0
- joint left_wheel2_joint: origin xyz=0.1 0.22 0 rpy=-1.5707 0 0 -> xyz=0.07 0.154 0 rpy=-1.5707 0 0
- joint lidar_joint: origin xyz=0 0 0.54 rpy=0 0 0 -> xyz=0 0 0.39 rpy=0 0 0
- joint right_wheel1_joint: origin xyz=-0.1 -0.22 0 rpy=-1.5707 0 0 -> xyz=-0.07 -0.154 0 rpy=-1.5707 0 0
- joint right_wheel2_joint: origin xyz=0.1 -0.22 0 rpy=-1.5707 0 0 -> xyz=0.07 -0.154 0 rpy=-1.5707 0 0

Commit message: nav server and client corrected, now using nav2 for planned paths/explored and odometery blind move when unexplored destination

File: install/r2d2_main/share/r2d2_main/urdf/robot.urdf (robot description, URDF)
Before this commit: robot r2d2, 8 links, 7 joints
Joints:
- joint camera_joint: origin xyz=0.05 0 0 rpy=0 0 0 -> xyz=0.03 0 0 rpy=0 0 0
